File: boards/ledecorator-core-board/ledecorator-core-board.brd (EAGLE design)
At the start: 50 x 100 mm, 69 parts, among them IC1 DS1307Z, IC1(CORE) ATMEGA48/88/168-PU, IC1(DISPLAY) ATMEGA48/88/168-PU, J1 DCJ0202, Q1 20MHz, Q2 20MHz, Q3 32KHz, Q4 BC557, Q5 BC557, T1 2SC1815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

Commit message: CORE: board
Parts:
- removed C16: (no value), rcl:E2-4
- removed JP3: (no value), pinhead:1X05/90
- removed R24, R25, R27: (no value), rcl:R1206
- added C13: (no value), rcl:C1206
- added JP4: (no value), pinhead:1X05
- added R19: (no value), rcl:0207/10
- added R5, R6: (no value), rcl:0207/12
- C14: value 10u -> (none); device rcl:E2-4 -> rcl:C050-025X075
- C4, C6: device rcl:C025-025X050 -> rcl:C1206
- R1: value 10K -> 10k
- R10, R12, R13, R14, R15, R16, R17, R18, R9: device rcl:R1206 -> rcl:0207/10
- R11: device rcl:R1206 -> rcl:0207/12
- R3: value 4.7K -> 4.7k; device rcl:0207/10 -> rcl:R1206
- R4: device rcl:0207/10 -> rcl:R1206
- moved R18 692.4 mm to (19.2, 134.8)
- moved R26 662.5 mm to (19.8, 83.2), flipped to the bottom, turned to 270 degrees
- moved R23 649.2 mm to (23.2, 83.2), flipped to the bottom, turned to 270 degrees
- moved R17 631.4 mm to (10.0, 78.8)
- moved R10 621.1 mm to (47.5, 89.8), turned to 180 degrees
- moved R11 616.8 mm to (22.0, 89.5), turned to 180 degrees
- moved R9 613.4 mm to (47.5, 86.5), turned to 180 degrees
- moved R12 597.7 mm to (20.0, 65.0), turned to 90 degrees
- moved R8 597.1 mm to (30.0, 80.8), flipped to the bottom
- moved R7 589.2 mm to (30.0, 77.2), flipped to the bottom
- moved R14 585.8 mm to (30.2, 38.5), turned to 90 degrees
- moved R16 581.9 mm to (33.0, 23.2), turned to 180 degrees
- moved R13 580.1 mm to (27.5, 38.5), turned to 90 degrees
- moved R15 574.4 mm to (33.0, 20.2), turned to 180 degrees
- moved U$8 565.1 mm to (3.75, 71.8), turned to 90 degrees
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Connections:
- net N$27 renamed SCL
- net N$32 renamed DISPLAY$TX
- net N$33 renamed TX
- net N$38 renamed BLE$TX
- net N$41 renamed USB$STATE
- net N$44 renamed BLE$RX
- net N$47 renamed USB$TX
- net N$48 renamed USB$RX
- net N$5 renamed DISPLAY$RX
- removed net N$14: IC1.2, Q3.1
- removed net N$24: IC1(CORE).25, R13.1, R14.1
- removed net N$39: R20.2, U$3.1
- removed net N$40: C14.+, IC1(CORE).5, R20.1
- removed net N$46: C16.+, IC1(CORE).26, R23.1, R24.1, R25.1, R26.1, R27.2
- removed net N$84: IC1(CORE).2, R11.1, R15.1, R7.1, T1.E, T3.E, T5.E
- new net BLE$CTRL: IC1(CORE).13, R15.1, R16.1
- new net BLR$STATE$1: C13.1, IC1(CORE).5, R20.1
- new net DISPLAY$SRC: C14.1, IC1(CORE).26, R17.2, R18.1, R19.1, R23.1, R26.1
- new net N$5: IC1.2, Q3.2
- new net RX: IC1(CORE).2, R11.1, R5.1, R7.1, T1.E, T3.E, T5.E
- new net USB$CTRL: IC1(CORE).12, R13.1, R14.1
- net +5V: now also JP4.2, R5.2, R6.2; no longer JP3.1, R15.2, R16.2
- net GND: now also C13.2, C14.2, JP4.1, R4.1; no longer C14.-, C16.-, JP3.2
- net N$1: now also C6.1; no longer C4.1
- net N$12: no longer R4.1
- net N$13: now also Q3.1; no longer Q3.2
- net N$19: now also R15.2; no longer R17.2
- net N$20: now also R16.2; no longer R18.2
- net N$21: now also R20.2, U$3.6; no longer IC1(CORE).24, R17.1, R18.1
- net N$25: now also R18.2; no longer R24.2
- net N$26: now also R19.2; no longer R25.2
- net N$28: now also R6.1; no longer R16.1
- net N$29: now also JP4.5; no longer JP3.5
- net N$51: now also JP4.3; no longer JP3.3
- net N$53: now also R17.1; no longer R27.1
- net N$6: now also C4.1; no longer C6.1
- net SCK: now also JP4.4; no longer JP3.4
Routing:
- net GND: track 0.00 -> 656.3 mm, vias 0 -> 6
- net +5V: track 0.00 -> 475.1 mm, vias 0 -> 4
- net TX: track 0.00 -> 161.2 mm, vias 0 -> 4
- net RESET: track 0.00 -> 145.0 mm, vias 0 -> 4
- net DISPLAY$SRC: track 0.00 -> 140.0 mm, vias 0 -> 2
- net SCK: track 0.00 -> 139.2 mm, vias 0 -> 6
- net RX: track 0.00 -> 130.6 mm, vias 0 -> 4
- net DISPLAY$RX: track 0.00 -> 119.1 mm
- net SCL: track 0.00 -> 113.9 mm
- net SDA: track 0.00 -> 111.5 mm
- net DISPLAY$TX: track 0.00 -> 89.7 mm
- net BLR$STATE$1: track 0.00 -> 86.7 mm
- net N$37: track 0.00 -> 84.8 mm, vias 0 -> 2
- net N$28: track 0.00 -> 81.8 mm
- net BLE$TX: track 0.00 -> 72.1 mm
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- added copper zone on layer 16, net GND
Other:
- board size 50 x 100 mm -> 60 x 150 mm
- board text added: "DISPLAY"
- board text added: "DRAGBERRY"
- board text added: "GND VCC DATA CLCK CTRL"
- board text added: "LEDECORATOR"
- board text added: "MISO MOSI"
- board text added: "RESET MOSI MISO SCK"

Commit message: Core: fix board
Parts:
- removed R17: (no value), rcl:0207/10
- added U$6: (no value), dragberry:SS12D00
- C13, C14: value (none) -> 1u
- JP1: device pinhead:1X04/90 -> pinhead:1X06/90
- R10, R13, R14, R15, R16, R18, R19, R23, R26, R9: value (none) -> 220
- R11, R12, R5, R6, R7, R8: value (none) -> 2k
- moved LED1 17.3 mm to (38.8, 13.4), turned to 180 degrees
- moved R4 11.1 mm to (46.5, 16.5)
- moved R3 5.77 mm to (46.5, 13.5)
- moved Q3 3.72 mm to (48.5, 8.75)
- moved JP1 3.72 mm to (4.50, 113.2)
- moved JP2 1.75 mm to (4.50, 62.5)
- moved U$4 1.50 mm to (55.8, 98.0)
- moved U$5 1.50 mm to (51.5, 98.0)
- moved R1 1.12 mm to (37.5, 87.2)
- moved T2 1.03 mm to (32.2, 95.5)
- moved R8 0.75 mm to (30.0, 80.0)
- moved T1 0.56 mm to (32.1, 86.2)
- moved R7 0.50 mm to (30.0, 76.8)
Connections:
- removed net N$15: LED1.K, R4.2
- removed net N$53: R17.1, U$8.P$2
- new net N$14: IC1.7, LED1.K, R3.1
- new net SCK$CORE: IC1(CORE).19, U$6.1$O
- new net SCK$DISPLAY: IC1(DISPLAY).19, JP4.4, U$6.1$S
- net +5V: now also JP1.5, R4.2; no longer LED1.A
- net DISPLAY$SRC: now also U$8.P$2; no longer R17.2
- net GND: now also JP1.6; no longer R4.1
- net MOSI: now also JP1.1; no longer JP1.3
- net N$11: now also LED1.A, R4.1; no longer IC1.7, R3.1
- net SCK: now also JP1.3, U$6.1$P; no longer IC1(CORE).19, IC1(DISPLAY).19, JP1.1, JP4.4
Routing:
- net SCK: track 139.2 -> 51.7 mm, vias 6 -> 2
- net SCK$DISPLAY: track 0.00 -> 54.9 mm, vias 0 -> 2
- net SCK$CORE: track 0.00 -> 48.1 mm, vias 0 -> 2
- net MISO: track 69.9 -> 50.6 mm
- net DISPLAY$SRC: track 140.0 -> 157.8 mm, vias 2 -> 4
- net N$14: track 0.00 -> 15.6 mm
- net MOSI: track 66.5 -> 53.1 mm
- net N$53: track 9.13 -> 0.00 mm
- net N$12: track 16.1 -> 22.3 mm
- net RESET: track 145.0 -> 150.9 mm
- net GND: track 656.3 -> 653.0 mm
- net +5V: track 475.1 -> 478.5 mm
- net N$15: track 3.26 -> 0.00 mm
- net N$11: track 8.05 -> 6.27 mm
- net N$49: track 56.7 -> 58.3 mm
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Other:
- board text added: "GND VCC RESET SCK MISO MOSI"
- board text removed: "MISO MOSI"
- board text removed: "RESET MOSI MISO SCK"
