File: boards/ledecorator-core-board/ledecorator-core-board.sch (EAGLE design)
At the start: 69 parts, among them IC1 DS1307Z, IC1(CORE) ATMEGA48/88/168-PU, IC1(DISPLAY) ATMEGA48/88/168-PU, J1 DCJ0202, Q1 20MHz, Q2 20MHz, Q3 32KHz, Q4 BC557, Q5 BC557, T1 2SC1815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

Commit message: CORE: board
Parts:
- removed C16: (no value), rcl:CPOL-EUE2-4
- removed JP3: (no value), pinhead:PINHD-1X5/90
- removed R24, R25, R27: (no value), rcl:R-EU_R1206
- added C13: (no value), rcl:C-EUC1206
- added JP4: (no value), pinhead:PINHD-1X5
- added R19: (no value), rcl:R-EU_0207/10
- added R5, R6: (no value), rcl:R-EU_0207/12
- C14: value 10u -> (none); device rcl:CPOL-EUE2-4 -> rcl:C-EU050-025X075
- C4, C6: device rcl:C-EU025-025X050 -> rcl:C-EUC1206
- R1: value 10K -> 10k
- R10, R12, R13, R14, R15, R16, R17, R18, R9: device rcl:R-EU_R1206 -> rcl:R-EU_0207/10
- R11: device rcl:R-EU_R1206 -> rcl:R-EU_0207/12
- R3: value 4.7K -> 4.7k; device rcl:R-EU_0207/10 -> rcl:R-EU_R1206
- R4: device rcl:R-EU_0207/10 -> rcl:R-EU_R1206
Connections:
- net N$27 renamed SCL
- net N$32 renamed DISPLAY$TX
- net N$33 renamed TX
- net N$38 renamed BLE$TX
- net N$41 renamed USB$STATE
- net N$44 renamed BLE$RX
- net N$47 renamed USB$TX
- net N$48 renamed USB$RX
- net N$5 renamed DISPLAY$RX
- removed net N$14: IC1.X2, Q3.1
- removed net N$24: IC1(CORE).PC2(ADC2/PCINT10), R13.1, R14.1
- removed net N$39: R20.2, U$3.STATE
- removed net N$40: C14.+, IC1(CORE).PD3(INT1/OC2B/PCINT19), R20.1
- removed net N$46: C16.+, IC1(CORE).PC3(ADC3/PCINT11), R23.1, R24.1, R25.1, R26.1, R27.2
- removed net N$84: IC1(CORE).PD0(RXD/PCINT16), R11.1, R15.1, R7.1, T1.E, T3.E, T5.E
- new net BLE$CTRL: IC1(CORE).PD7(AIN1/PCINT23), R15.1, R16.1
- new net BLR$STATE$1: C13.1, IC1(CORE).PD3(INT1/OC2B/PCINT19), R20.1
- new net DISPLAY$SRC: C14.1, IC1(CORE).PC3(ADC3/PCINT11), R17.2, R18.1, R19.1, R23.1, R26.1
- new net N$5: IC1.X2, Q3.2
- new net RX: IC1(CORE).PD0(RXD/PCINT16), R11.1, R5.1, R7.1, T1.E, T3.E, T5.E
- new net USB$CTRL: IC1(CORE).PD6(AIN0/OC0A/PCINT22), R13.1, R14.1
- net +5V: now also JP4.2, R5.2, R6.2; no longer JP3.1, R15.2, R16.2
- net GND: now also C13.2, C14.2, JP4.1, R4.1; no longer C14.-, C16.-, JP3.2
- net N$1: now also C6.1; no longer C4.1
- net N$12: no longer R4.1
- net N$13: now also Q3.1; no longer Q3.2
- net N$19: now also R15.2; no longer R17.2
- net N$20: now also R16.2; no longer R18.2
- net N$21: now also R20.2, U$3.EN; no longer IC1(CORE).PC1(ADC1/PCINT9), R17.1, R18.1
- net N$25: now also R18.2; no longer R24.2
- net N$26: now also R19.2; no longer R25.2
- net N$28: now also R6.1; no longer R16.1
- net N$29: now also JP4.5; no longer JP3.5
- net N$51: now also JP4.3; no longer JP3.3
- net N$53: now also R17.1; no longer R27.1
- net N$6: now also C4.1; no longer C6.1
- net SCK: now also JP4.4; no longer JP3.4
Other:
- moved on the sheet: C4, C6, G1, Q3, R15, R16, R17, R18, R4

Commit message: Core: fix board
Parts:
- removed R17: (no value), rcl:R-EU_0207/10
- added U$6: (no value), dragberry:SS12D00DIP
- C13, C14: value (none) -> 1u
- JP1: device pinhead:PINHD-1X4/90 -> pinhead:PINHD-1X6/90
- R10, R13, R14, R15, R16, R18, R19, R23, R26, R9: value (none) -> 220
- R11, R12, R5, R6, R7, R8: value (none) -> 2k
Connections:
- removed net N$15: LED1.C, R4.2
- removed net N$53: R17.1, U$8.P
- new net N$14: IC1.SQW, LED1.C, R3.1
- new net SCK$CORE: IC1(CORE).PB5(SCK/PCINT5), U$6.O
- new net SCK$DISPLAY: IC1(DISPLAY).PB5(SCK/PCINT5), JP4.4, U$6.S
- net +5V: now also JP1.5, R4.2; no longer LED1.A
- net DISPLAY$SRC: now also U$8.P; no longer R17.2
- net GND: now also JP1.6; no longer R4.1
- net MOSI: now also JP1.1; no longer JP1.3
- net N$11: now also LED1.A, R4.1; no longer IC1.SQW, R3.1
- net SCK: now also JP1.3, U$6.P; no longer IC1(CORE).PB5(SCK/PCINT5), IC1(DISPLAY).PB5(SCK/PCINT5), JP1.1, JP4.4
Other:
- moved on the sheet: LED1, R3, R4
